Commit message: added wheels

File: sim_tutorial/description/urdf/inertias.xacro (robot description, xacro)
@@ -14,3 +14,11 @@
     <!-- NOTE: wheels are radially symmetric around the x-axis -->
     <!-- TODO: define a macro for the inertial of a wheel (can approx as a cylinder) -->
+    <xacro:macro name="wheel_inertial" params="m r h">
+        <mass value="${m}"/>
+        <inertia
+            ixx="${m*r*r/2}" ixy="0" ixz="0"
+            iyy="${m*(2*r*r + h*h)/12}" iyz="0"
+            izz="${m*(2*r*r + h*h)/12}"
+        />
+    </xacro:macro>
 </robot>
