Commit message: added controller

File: sim_tutorial/description/urdf/cybertruck.urdf.xacro (robot description, xacro)
@@ -4,4 +4,5 @@
   <xacro:include filename="$(find description)/urdf/constants.xacro"/>
   <xacro:include filename="$(find description)/urdf/inertias.xacro"/>
+  <xacro:include filename="$(find description)/urdf/plugins.gazebo.xacro"/>
   <link name="base_link"/>
   <!-- Your URDF code here -->
@@ -19,14 +20,4 @@
         <mesh filename="package://description/urdf/meshes/cybertruck_body.dae"/>
       </geometry>
-    <!-- Motor Transmissions -->
-    <xacro:macro name="Transmission" params="joint">
-        <transmission name="${joint}_trans">
-            <type>transmission_interface/SimpleTransmission</type>
-            <joint name="${joint}">
-                <hardwareInterface>hardware_interface/EffortJointInterface</hardwareInterface>
-            </joint>
-            <actuator name="${joint}_motor"/>
-        </transmission>
-    </xacro:macro>
     </collision>
     <inertial>
@@ -41,3 +32,10 @@
   <!-- Wheels -->
   <xacro:include filename="$(find description)/urdf/wheels.urdf.xacro"/>
+  <!-- LIDAR -->
+  <link name="scan_link"/>
+  <joint name="scan_joint" type="fixed">
+    <parent link="body_link"/>
+    <child link="scan_link"/>
+    <origin xyz="0 ${front_wheel} ${-height_to_wheel}" rpy="0 0 ${-pi / 2}"/>
+  </joint>
 </robot>

File: sim_tutorial/description/urdf/inertias.xacro (robot description, xacro)
@@ -18,6 +18,6 @@
         <inertia
             ixx="${m*r*r/2}" ixy="0" ixz="0"
-            iyy="${m*(2*r*r + h*h)/12}" iyz="0"
-            izz="${m*(2*r*r + h*h)/12}"
+            iyy="${m*(3*r*r + h*h)/12}" iyz="0"
+            izz="${m*(3*r*r + h*h)/12}"
         />
     </xacro:macro>

File: sim_tutorial/description/urdf/wheels.urdf.xacro (robot description, xacro)
@@ -4,4 +4,14 @@
     <xacro:include filename="$(find description)/urdf/constants.xacro"/>
     <xacro:include filename="$(find description)/urdf/inertias.xacro"/>
+    <!-- Motor Transmissions -->
+    <xacro:macro name="Transmission" params="joint">
+        <transmission name="${joint}_trans">
+            <type>transmission_interface/SimpleTransmission</type>
+            <joint name="${joint}">
+                <hardwareInterface>hardware_interface/EffortJointInterface</hardwareInterface>
+            </joint>
+            <actuator name="${joint}_motor"/>
+        </transmission>
+    </xacro:macro>
     <!-- Wheel macro -->
     <xacro:macro name="Wheel" params="fb lr">
@@ -31,5 +41,4 @@
             <axis xyz="1 0 0"/>
         </joint>
-        <!-- Other attributes-->
         <xacro:if value="${fb == 'front'}">
             <!-- Add Transmission to Wheels connected to the motor -->
